File: Hardware/Panel/arpenvfol_panel/arpenvfol_panel.kicad_sch (KiCad schematic)
At the start: 16 parts, among them J4 mic_pad

Commit message: schem tweak
Parts:
- GRAF1: footprint (none) -> arpenvfol_panel:arpenvfol_panel_holes
- GRAF2: footprint (none) -> arpenvfol_panel:arpenvfol_panel_art
- J1: value (none) -> mic_hole; footprint (none) -> ao_tht:TestPoint_THTPad_1.5x1.5mm_Drill0.7mm
- J2: value (none) -> mic_hole; footprint (none) -> ao_tht:TestPoint_THTPad_D1.5mm_Drill0.7mm
- J3: value (none) -> mic_pad; footprint (none) -> TestPoint:TestPoint_Pad_D4.0mm
Other:
- title: (none) -> ARP envelope follower panel
Changed lines of the file:
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@@
   (paper "USLetter")
   (title_block
+    (title "ARP envelope follower panel")
+    (date "2022-03-27")
     (company "Rich Holmes / Analog Output")
     (comment 1 "or neighboring rights to this work. Published from United States.")
@@
       (effects (font (size 1.27 1.27)) (justify left))
     )
-    (property "Footprint" "" (id 2) (at 175.26 50.8 0)
+    (property "Footprint" "arpenvfol_panel:arpenvfol_panel_holes" (id 2) (at 175.26 50.8 0)
       (effects (font (size 1.27 1.27)) hide)
     )
@@
       (effects (font (size 1.27 1.27)) (justify left))
     )
-    (property "Footprint" "" (id 2) (at 175.26 57.15 0)
+    (property "Footprint" "arpenvfol_panel:arpenvfol_panel_art" (id 2) (at 175.26 57.15 0)
       (effects (font (size 1.27 1.27)) hide)
     )
@@
     (in_bom yes) (on_board yes) (fields_autoplaced)
     (property "Reference" "J2" (id 0) (at 127 58.5302 0))
-    (property "Value" "" (id 1) (at 127 61.0671 0))
-    (property "Footprint" "" (id 2) (at 127 63.5 0)
+    (property "Value" "mic_hole" (id 1) (at 127 61.0671 0))
+    (property "Footprint" "ao_tht:TestPoint_THTPad_D1.5mm_Drill0.7mm" (id 2) (at 127 63.5 0)
       (effects (font (size 1.27 1.27)) hide)
     )
@@
     (in_bom yes) (on_board yes) (fields_autoplaced)
     (property "Reference" "J1" (id 0) (at 127 45.8302 0))
-    (property "Value" "" (id 1) (at 127 48.3671 0))
-    (property "Footprint" "" (id 2) (at 127 50.8 0)
+    (property "Value" "mic_hole" (id 1) (at 127 48.3671 0))
+    (property "Footprint" "ao_tht:TestPoint_THTPad_1.5x1.5mm_Drill0.7mm" (id 2) (at 127 50.8 0)
       (effects (font (size 1.27 1.27)) hide)
     )
@@
       (effects (font (size 1.27 1.27)) (justify left))
     )
-    (property "Value" "" (id 1) (at 139.192 52.5022 0)
-      (effects (font (size 1.27 1.27)) (justify left))
-    )
-    (property "Footprint" "" (id 2) (at 137.16 50.8 0)
-      (effects (font (size 1.27 1.27)) hide)
-    )
+    (property "Value" "mic_pad" (id 1) (at 139.192 52.5022 0)
+      (effects (font (size 1.27 1.27)) (justify left))
+    )
+    (property "Footprint" "TestPoint:TestPoint_Pad_D4.0mm" (id 2) (at 137.16 50.8 0)
+      (effects (font (size 1.27 1.27)) hide)
+    )
