File: Hardware/Panel/arpenvfol_panel/arpenvfol_panel.kicad_pcb (KiCad board)
At the start: 2 copper layers, 50 x 200 mm, 16 parts, among them J1 mic_hole, J2 mic_hole, J3 mic_pad, J4 mic_pad

Commit message: Final pre fab tweaks, Gerbers, schematic, BOM
Parts:
- moved J1 2.50 mm to (29.9, 134.6)
- moved J2 2.50 mm to (27.4, 134.6)
Other:
- board text added: "Ground"
- board text added: "Panel design by Rich Holmes CC0 1.0 Mar 2022 JLCJLCJLCJLC"
- board text removed: "Panel design by Rich Holmes CC0 1.0 Mar 2021 JLCJLCJLCJLC"
Changed lines of the file:
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@@
   )
   (footprint "ao_tht:TestPoint_THTPad_D1.5mm_Drill0.7mm" (layer "F.Cu")
-    (at 29.85 134.6)
+    (at 27.35 134.6)
     (descr "THT pad as test Point, diameter 1.5mm, hole diameter 0.7mm")
     (tags "test point THT pad")
@@
   )
   (footprint "ao_tht:TestPoint_THTPad_1.5x1.5mm_Drill0.7mm" (layer "F.Cu")
-    (at 27.35 134.6)
+    (at 29.85 134.6)
     (descr "THT rectangular pad as test Point, square 1.5mm side length, hole diameter 0.7mm")
     (tags "test point THT pad rectangle square")
@@
     (fp_circle (center 0 0) (end 0 -2.25) (layer "B.SilkS") (width 0.12) (fill none))
     (fp_circle (center 0 0) (end 2.5 0) (layer "B.CrtYd") (width 0.05) (fill none))
-    (pad "1" smd circle (at 0 0) (size 4 4) (layers "B.Cu" "B.Mask")
+    (pad "1" smd circle (at -11 0) (size 4 4) (layers "B.Cu" "B.Mask")
       (net 2 "Net-(J2-Pad1)") (pinfunction "Pin_1") (pintype "passive"))
   )
@@
     (fp_circle (center 0 0) (end 0 -2.25) (layer "B.SilkS") (width 0.12) (fill none))
     (fp_circle (center 0 0) (end 2.5 0) (layer "B.CrtYd") (width 0.05) (fill none))
-    (pad "1" smd circle (at 0 0) (size 4 4) (layers "B.Cu" "B.Mask")
+    (pad "1" smd circle (at 11 0) (size 4 4) (layers "B.Cu" "B.Mask")
       (net 1 "GND") (pinfunction "Pin_1") (pintype "passive"))
   )
@@
     (effects (font (size 1 1) (thickness 0.15)) (justify mirror))
   )
+  (gr_text "Ground" (at 34.1 137.85) (layer "B.SilkS")
+    (effects (font (size 1 1) (thickness 0.15)) (justify mirror))
+  )
   (gr_text "Synth in" (at 53.6 142.6) (layer "B.SilkS")
     (effects (font (size 1 1) (thickness 0.15)) (justify mirror))
@@
     (effects (font (size 1 1) (thickness 0.15)) (justify mirror))
   )
-  (gr_text "Panel design by Rich Holmes\nCC0 1.0 Mar 2021\nJLCJLCJLCJLC" (at 41.1 197.6) (layer "B.SilkS")
+  (gr_text "Panel design by Rich Holmes\nCC0 1.0 Mar 2022\nJLCJLCJLCJLC" (at 41.1 197.6) (layer "B.SilkS")
     (effects (font (size 1 1) (thickness 0.15)) (justify mirror))
   )
@@
     (effects (font (size 1 1) (thickness 0.15)) (justify mirror))
   )
-  (segment (start 23.1 134.6) (end 27.35 134.6) (width 0.25) (layer "B.Cu") (net 1))
-  (segment (start 29.85 134.6) (end 34.1 134.6) (width 0.25) (layer "B.Cu") (net 2))
+  (segment (start 29.85 134.6) (end 34.1 134.6) (width 0.25) (layer "B.Cu") (net 1))
+  (segment (start 23.1 134.6) (end 27.35 134.6) (width 0.25) (layer "B.Cu") (net 2))
   (zone (net 1) (net_name "GND") (layers F&B.Cu) (hatch edge 0.508)
     (connect_pads (clearance 0.508))
